Commit message: mannaggia

File: src/naaut-base/urdf/robot.urdf (robot description, URDF)
Before this commit: robot diglobot2, 6 links, 5 joints
Links:
- removed link base_footprint
- removed link fwheel
- removed link lwheel
- removed link rwheel
- added link base_link; visual box size=0.48 0.3 0.01
- added link gps_link; visual box size=0.05 0.05 0.05
- added link lfloater; visual cylinder length=2.8 radius=0.18
- added link rfloater; visual cylinder length=2.8 radius=0.18
Joints:
- removed joint base_to_fwheel
- removed joint base_to_lwheel
- removed joint base_to_rwheel
- added joint base_to_lfloater: type fixed, parent base_link, child lfloater, origin xyz=0 0.8 0.085 rpy=1.5708 0 1.5708
- added joint base_to_rfloater: type fixed, parent base_link, child rfloater, origin xyz=0 -0.8 0.085 rpy=-1.5708 0 1.5708
- added joint gps_joint: type fixed, parent base_link, child gps_link, origin xyz=0.21 -0.02 0.35 rpy=0 0 0
- joint base_to_scanner: origin xyz=0.045 0 0.225 rpy=0 0 -1.57079 -> xyz=0.045 0 1.0 rpy=0 0 -1.57079; parent base_footprint -> base_link
- joint imu_joint: parent base_footprint -> base_link
